File: Hardware/SparkFun_GPS_ZED-F9K.brd (EAGLE design)
At the start: 43.2 x 43.2 mm, 104 parts, among them J1 QWIIC_RIGHT_ANGLE, J4 U.FL, J6 QWIIC_RIGHT_ANGLE, U2 3.3V, U3 UBLOX_ZED_F9K, U4 TRIPLE_BUFFER_74LVC3G07

Commit message: Fixes labels on BoB
Parts:
- removed U$44: (no value), more_all_labels:SCL#CLK3
- added U$59: (no value), Labels:CS#-[>-04
- U$24: device ALL_LABELS:INT1 -> bottom labels:INT2
- U$27: device ALL_LABELS:PPS4 -> bottom labels:PPS1
- U$28: device ALL_LABELS:SAFEBOOT2 -> bottom labels:RESET4
- U$30: device moar:RESET0 -> corrected_bottom:RXI#MOSI0
- U$32: device Labels:CS#-[>-04 -> bottom labels:SAFEBOOT3
- U$37: device Labels:SCL-[) -> corrected_bottom:TXO#MISO1
- U$38: device Labels:SDA-[) -> corrected_bottom:SCL#CLK2
- U$39: device more_all_labels:TXR0 -> corrected_bottom:SCL5
- U$42: device more_all_labels:RXI#MOSI1 -> corrected_bottom:SDA4
- U$43: device more_all_labels:TXO#MISO2 -> corrected_bottom:TXR3
- moved U$38 42.0 mm to (41.7, 14.0), turned to 0 degrees
- moved U$37 41.9 mm to (41.7, 16.5), turned to 0 degrees
- moved U$30 40.7 mm to (41.7, 19.1), turned to 0 degrees
- moved U$32 31.3 mm to (11.3, 13.8)
- moved U$42 27.9 mm to (6.35, 26.7), turned to 0 degrees
- moved U$43 26.0 mm to (6.48, 18.9), turned to 0 degrees
- moved U$39 11.1 mm to (6.10, 29.2), turned to 0 degrees
- moved U$28 6.93 mm to (8.13, 11.4), turned to 0 degrees
- moved U$34 4.95 mm to (34.3, 36.7), turned to 90 degrees
- moved U$27 4.46 mm to (6.10, 8.89), turned to 0 degrees
- moved U$24 4.33 mm to (5.84, 16.5), turned to 0 degrees
- moved U$35 0.13 mm to (26.7, 36.7)
Changed lines of the file:
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@@
 <layer number="45" name="Holes" color="7" fill="1" visible="yes" active="yes"/>
 <layer number="46" name="Milling" color="3" fill="1" visible="no" active="yes"/>
-<layer number="47" name="Measures" color="7" fill="1" visible="yes" active="yes"/>
+<layer number="47" name="Measures" color="7" fill="1" visible="no" active="yes"/>
 <layer number="48" name="Document" color="7" fill="1" visible="no" active="yes"/>
 <layer number="49" name="Reference" color="13" fill="1" visible="yes" active="yes"/>
@@
 <layer number="115" name="ReferenceISLANDS" color="7" fill="1" visible="no" active="no"/>
 <layer number="116" name="Patch_BOT" color="9" fill="4" visible="no" active="no"/>
-<layer number="117" name="PM_Ref" color="26" fill="1" visible="yes" active="yes"/>
+<layer number="117" name="PM_Ref" color="26" fill="1" visible="no" active="yes"/>
 <layer number="118" name="Rect_Pads" color="7" fill="1" visible="no" active="no"/>
-<layer number="119" name="PF_Ref" color="31" fill="1" visible="yes" active="yes"/>
-<layer number="120" name="WFL_Ref" color="25" fill="1" visible="yes" active="yes"/>
+<layer number="119" name="PF_Ref" color="31" fill="1" visible="no" active="yes"/>
+<layer number="120" name="WFL_Ref" color="25" fill="1" visible="no" active="yes"/>
 <layer number="121" name="_tsilk" color="7" fill="1" visible="no" active="no"/>
 <layer number="122" name="_bsilk" color="7" fill="1" visible="no" active="no"/>
@@
 <element name="U$21" library="TXR" package="BLK2" value="" x="34.798" y="41.91" smashed="yes"/>
 <element name="U$23" library="TXR" package="GRN1" value="" x="17.399" y="42.037" smashed="yes"/>
-<element name="U$24" library="ALL_LABELS" package="INT1" value="" x="1.508" y="16.513" smashed="yes" rot="MR180"/>
-<element name="U$27" library="ALL_LABELS" package="PPS4" value="" x="1.635" y="8.873" smashed="yes" rot="MR180"/>
-<element name="U$28" library="ALL_LABELS" package="SAFEBOOT2" value="" x="1.635" y="13.856" smashed="yes" rot="MR180"/>
-<element name="U$30" library="moar" package="RESET0" value="" x="1.635" y="11.403" smashed="yes" rot="MR180"/>
-<element name="U$37" library="Labels" package="SCL-[)" value="" x="1.651" y="29.1084" smashed="yes" rot="MR180"/>
-<element name="U$38" library="Labels" package="SDA-[)" value="" x="1.651" y="26.67" smashed="yes" rot="MR180"/>
 <element name="U$40" library="Labels" package="3V3-04" value="" x="6.223" y="24.13" smashed="yes" rot="MR0"/>
 <element name="U$41" library="Labels" package="GND-04" value="" x="6.477" y="21.5646" smashed="yes" rot="MR0"/>
 <element name="U$29" library="Labels" package="3V3-04" value="" x="41.656" y="24.13" smashed="yes" rot="MR0"/>
 <element name="U$31" library="Labels" package="GND-04" value="" x="41.529" y="29.1846" smashed="yes" rot="MR0"/>
-<element name="U$32" library="Labels" package="CS#-[&gt;-04" value="" x="41.656" y="21.463" smashed="yes" rot="MR0"/>
 <element name="U$33" library="Labels" package="5V" value="" x="41.656" y="26.67" smashed="yes" rot="MR0"/>
-<element name="U$34" library="Labels" package="GND-04" value="" x="34.29" y="41.656" smashed="yes" rot="MR270"/>
-<element name="U$35" library="ALL_LABELS" package="RXI28" value="" x="26.67" y="36.576" smashed="yes" rot="MR90"/>
+<element name="U$34" library="Labels" package="GND-04" value="" x="34.29" y="36.703" smashed="yes" rot="MR90"/>
+<element name="U$35" library="ALL_LABELS" package="RXI28" value="" x="26.67" y="36.703" smashed="yes" rot="MR90"/>
 <element name="U$36" library="moar" package="TXO21" value="" x="24.13" y="35.814" smashed="yes" rot="MR90"/>
-<element name="U$39" library="more_all_labels" package="TXR0" value="" x="1.651" y="19.05" smashed="yes" rot="MR180"/>
-<element name="U$42" library="more_all_labels" package="RXI#MOSI1" value="" x="33.147" y="18.923" smashed="yes" rot="MR180"/>
-<element name="U$43" library="more_all_labels" package="TXO#MISO2" value="" x="32.385" y="16.51" smashed="yes" rot="MR180"/>
-<element name="U$44" library="more_all_labels" package="SCL#CLK3" value="" x="33.655" y="13.97" smashed="yes" rot="MR180"/>
 <element name="U$45" library="more_all_labels" package="SPI4" value="" x="11.811" y="16.891" smashed="yes" rot="MR0"/>
 <element name="U$46" library="Labels" package="I_SUPER2_C-()-04" value="" x="10.033" y="23.241" smashed="yes" rot="MR0"/>
@@
 <element name="U$53" library="TXR" package="GRN1" value="" x="21.082" y="42.037" smashed="yes" rot="MR0"/>
 <element name="U$54" library="TXR" package="BLK2" value="" x="38.1" y="41.91" smashed="yes" rot="MR0"/>
+<element name="U$24" library="bottom labels" package="INT2" value="" x="5.842" y="16.51" smashed="yes" rot="MR0"/>
+<element name="U$27" library="bottom labels" package="PPS1" value="" x="6.096" y="8.89" smashed="yes" rot="MR0"/>
+<element name="U$28" library="bottom labels" package="RESET4" value="" x="8.128" y="11.43" smashed="yes" rot="MR0"/>
+<element name="U$32" library="bottom labels" package="SAFEBOOT3" value="" x="11.303" y="13.843" smashed="yes" rot="MR0"/>
+<element name="U$59" library="Labels" package="CS#-[&gt;-04" value="" x="41.783" y="21.59" smashed="yes" rot="MR0"/>
+<element name="U$30" library="corrected_bottom" package="RXI#MOSI0" value="" x="41.656" y="19.05" smashed="yes" rot="MR0"/>
+<element name="U$37" library="corrected_bottom" package="TXO#MISO1" value="" x="41.656" y="16.51" smashed="yes" rot="MR0"/>
+<element name="U$38" library="corrected_bottom" package="SCL#CLK2" value="" x="41.656" y="13.97" smashed="yes" rot="MR0"/>
+<element name="U$39" library="corrected_bottom" package="SCL5" value="" x="6.096" y="29.21" smashed="yes" rot="MR0"/>
+<element name="U$42" library="corrected_bottom" package="SDA4" value="" x="6.35" y="26.67" smashed="yes" rot="MR0"/>
+<element name="U$43" library="corrected_bottom" package="TXR3" value="" x="6.477" y="18.923" smashed="yes" rot="MR0"/>
 </elements>
 <signals>
