File: Hardware/SparkFun_GPS_ZED-F9K.sch (EAGLE design)
At the start: 48 parts, among them J1 QWIIC_RIGHT_ANGLE, J4 U.FL, J6 QWIIC_RIGHT_ANGLE, U2 3.3V, U3 UBLOX_ZED_F9K, U4 TRIPLE_BUFFER_74LVC3G07

Commit message: Fixes labels on BoB
Changed lines of the file:
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@@
+</nets>
+</sheet>
+<sheet>
+<plain>
+</plain>
+<instances>
+</instances>
+<busses>
+</busses>
+<nets>
+</nets>
+</sheet>
+<sheet>
+<plain>
+</plain>
+<instances>
+</instances>
+<busses>
+</busses>
+<nets>
 </nets>
 </sheet>
