File: Hardware/ZED-F9R_PhAT_v1.sch (EAGLE design)
At the start: 78 parts, among them J1 U.FL, J5 QWIIC_RIGHT_ANGLE, J6 RASPBERRYPI-40-PIN-GPIO_SMD_S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, U1 U-BLOX_ZED_F9R, U2 DUAL-OPTO_HCPL-073LSOIC-8, U3 UHS_INVERTER_SCHMITT_TRIGGER_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, U4 UHS_INVERTER_SCHMITT_TRIGGER_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

Commit message: Updates F9R module, Fixes various trace overlaps and acid traps
* Updates resistor values on LEDs
* Adds more capacitance to power lines
Parts:
- added C10: 1.0uF, SparkFun-Capacitors:1.0UF-0402-16V-10%
- added C9: 2.2uF, SparkFun-Capacitors:2.2UF-0402_TIGHT-10V-10%-X5R
- J2: device SparkFun-Connectors:USB_C_2-LAYER -> SparkFun-Connectors:USB_C_2-LAYER_PADS
- R10, R11, R12: value 4.7k -> 2.2k; device SparkFun-Resistors:4.7KOHM-0603-1/10W-1% -> SparkFun-Resistors:2.2KOHM-0603-1/10W-1%
- U1: value U-BLOX_ZED_F9R -> U-BLOX_ZED-F9R; device SparkFun-GPS:U-BLOX_ZED_F9R -> SparkFun-GPS:U-BLOX_ZED-F9R
Connections:
- net 3.3V: now also C10.1
- net GND: now also C10.2, C9.2
- net N$21: now also U1.TX/COPI; no longer U1.TX/MISO
- net N$26: now also U1.RX/CIPO; no longer U1.RX/MOSI
- net V_BATT: now also C9.1
Other:
- note added: "Dead Reckoning Module - u-blox ZED-F9R"
- note removed: "Dead Reckoning Module - ZED-F9R"
- moved on the sheet: C1, C2, C4, D1, D2, D3, JP1, JP2, JP3, R1, R10, R11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
