File: Hardware/Automotive Interface BoB/Automotive_Inter_BoB.brd (EAGLE design)
At the start: 25.4 x 25.4 mm, 49 parts, among them U1 HCPL-270L

Commit message: CAMs the Automotive Interface Board, updates parts in library with digikey links
Parts:
- C4, C5, C7: value 100nF -> 0.1uF; device classified:0603 -> SparkFun-Capacitors:0603
Changed lines of the file:
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@@
 <attribute name="VALUE" x="7.371" y="16.08166875" size="2.54" layer="27"/>
 </element>
-<element name="C5" library="classified" package="0603" value="100nF" x="17.653" y="22.606" smashed="yes" rot="R270">
+<element name="C5" library="SparkFun-Capacitors" package="0603" value="0.1uF" x="17.653" y="22.606" smashed="yes" rot="R270">
 <attribute name="NAME" x="18.415" y="22.606" size="0.6096" layer="25" font="vector" ratio="20" rot="R270" align="bottom-center"/>
-<attribute name="PROD_ID" value="" x="17.653" y="22.606" size="1.778" layer="27" font="vector" ratio="15" rot="R270" display="off"/>
-<attribute name="VALUE" x="16.891" y="22.606" size="0.6096" layer="27" font="vector" ratio="20" rot="R270" align="top-center"/>
+<attribute name="PROD_ID" value="CAP-08390" x="17.653" y="22.606" size="1.778" layer="27" font="vector" ratio="15" rot="R270" display="off"/>
+<attribute name="VALUE" value="0.1uF" x="16.891" y="22.606" size="0.6096" layer="27" font="vector" ratio="20" rot="R270" align="top-center"/>
 </element>
 <element name="J1" library="SparkFun-Connectors" package="1X06_NO_SILK" value="" x="1.27" y="6.35" smashed="yes" rot="R90">
@@
 <attribute name="VALUE" x="2.54" y="0.508" size="0.6096" layer="27" font="vector" ratio="20" align="top-center"/>
 </element>
-<element name="C4" library="classified" package="0603" value="100nF" x="22.352" y="17.272" smashed="yes" rot="R90">
+<element name="C4" library="SparkFun-Capacitors" package="0603" value="0.1uF" x="22.352" y="17.272" smashed="yes" rot="R90">
 <attribute name="NAME" x="21.59" y="17.272" size="0.6096" layer="25" font="vector" ratio="20" rot="R90" align="bottom-center"/>
-<attribute name="PROD_ID" value="" x="22.352" y="17.272" size="1.778" layer="27" font="vector" ratio="15" rot="R90" display="off"/>
-<attribute name="VALUE" x="23.114" y="17.272" size="0.6096" layer="27" font="vector" ratio="20" rot="R90" align="top-center"/>
+<attribute name="PROD_ID" value="CAP-08390" x="22.352" y="17.272" size="1.778" layer="27" font="vector" ratio="15" rot="R90" display="off"/>
+<attribute name="VALUE" value="0.1uF" x="23.114" y="17.272" size="0.6096" layer="27" font="vector" ratio="20" rot="R90" align="top-center"/>
 </element>
-<element name="C7" library="classified" package="0603" value="100nF" x="22.352" y="8.509" smashed="yes" rot="R90">
+<element name="C7" library="SparkFun-Capacitors" package="0603" value="0.1uF" x="22.352" y="8.509" smashed="yes" rot="R90">
 <attribute name="NAME" x="21.59" y="8.509" size="0.6096" layer="25" font="vector" ratio="20" rot="R90" align="bottom-center"/>
-<attribute name="PROD_ID" value="" x="22.352" y="8.509" size="1.778" layer="27" font="vector" ratio="15" rot="R90" display="off"/>
-<attribute name="VALUE" x="23.114" y="8.509" size="0.6096" layer="27" font="vector" ratio="20" rot="R90" align="top-center"/>
+<attribute name="PROD_ID" value="CAP-08390" x="22.352" y="8.509" size="1.778" layer="27" font="vector" ratio="15" rot="R90" display="off"/>
+<attribute name="VALUE" value="0.1uF" x="23.114" y="8.509" size="0.6096" layer="27" font="vector" ratio="20" rot="R90" align="top-center"/>
 </element>
 <element name="LOGO1" library="SparkFun-Aesthetics" package="SFE_LOGO_NAME_FLAME_.1" value="SFE_LOGO_NAME_FLAME.1_INCH" x="12.7" y="12.7" smashed="yes" rot="MR270"/>

Commit message: Adds wheel tick and direction circuit to pi-hat
Parts:
- moved C4 3.50 mm to (19.8, 19.7), turned to 180 degrees
Routing:
- net WT_OUT: track 8.28 -> 0.76 mm, vias 1 -> 0
- net 3.3V: track 55.9 -> 50.0 mm
- net DIR_OUT: track 4.23 -> 0.00 mm
Changed lines of the file:
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@@
 <?xml version="1.0" encoding="utf-8"?>
 <!DOCTYPE eagle SYSTEM "eagle.dtd">
-<eagle version="9.5.1">
+<eagle version="9.5.2">
 <drawing>
 <settings>
@@
 <layers>
 <layer number="1" name="Top" color="4" fill="1" visible="yes" active="yes"/>
+<layer number="2" name="Route2" color="1" fill="3" visible="no" active="yes"/>
+<layer number="15" name="Route15" color="4" fill="6" visible="no" active="yes"/>
 <layer number="16" name="Bottom" color="3" fill="1" visible="yes" active="yes"/>
 <layer number="17" name="Pads" color="26" fill="1" visible="yes" active="yes"/>
@@
 <attribute name="VALUE" x="2.54" y="0.508" size="0.6096" layer="27" font="vector" ratio="20" align="top-center"/>
 </element>
-<element name="C4" library="SparkFun-Capacitors" package="0603" value="0.1uF" x="22.352" y="17.272" smashed="yes" rot="R90">
-<attribute name="NAME" x="21.59" y="17.272" size="0.6096" layer="25" font="vector" ratio="20" rot="R90" align="bottom-center"/>
-<attribute name="PROD_ID" value="CAP-08390" x="22.352" y="17.272" size="1.778" layer="27" font="vector" ratio="15" rot="R90" display="off"/>
-<attribute name="VALUE" value="0.1uF" x="23.114" y="17.272" size="0.6096" layer="27" font="vector" ratio="20" rot="R90" align="top-center"/>
+<element name="C4" library="SparkFun-Capacitors" package="0603" value="0.1uF" x="19.812" y="19.685" smashed="yes" rot="R180">
+<attribute name="NAME" x="19.812" y="18.923" size="0.6096" layer="25" font="vector" ratio="20" rot="R180" align="bottom-center"/>
+<attribute name="PROD_ID" value="CAP-08390" x="19.812" y="19.685" size="1.778" layer="27" font="vector" ratio="15" rot="R180" display="off"/>
+<attribute name="VALUE" value="0.1uF" x="19.812" y="20.447" size="0.6096" layer="27" font="vector" ratio="20" rot="R180" align="top-center"/>
 </element>
 <element name="C7" library="SparkFun-Capacitors" package="0603" value="0.1uF" x="22.352" y="8.509" smashed="yes" rot="R90">
@@
 <contactref element="C4" pad="2"/>
 <contactref element="U$1" pad="P3"/>
+<wire x1="19.685" y1="16.256" x2="18.962" y2="19.685" width="0" layer="19" extent="1-1"/>
+<wire x1="18.534" y1="16.275" x2="19.685" y2="16.256" width="0" layer="19" extent="1-1"/>
+<wire x1="17.526" y1="19.685" x2="18.534" y2="16.275" width="0" layer="19" extent="1-1"/>
+<wire x1="17.653" y1="21.756" x2="17.526" y2="19.685" width="0" layer="19" extent="1-1"/>
+<wire x1="15.379" y1="19.812" x2="17.526" y2="19.685" width="0" layer="19" extent="1-1"/>
+<wire x1="15.24" y1="13.97" x2="18.534" y2="16.275" width="0" layer="19" extent="1-1"/>
+<wire x1="14.1605" y1="15.5135" x2="15.24" y2="13.97" width="0" layer="19" extent="1-1"/>
+<wire x1="15.24" y1="11.557" x2="15.24" y2="13.97" width="0" layer="19" extent="1-1"/>
+<wire x1="14.0335" y1="10.0135" x2="15.24" y2="11.557" width="0" layer="19" extent="1-1"/>
+<wire x1="18.534" y1="7.512" x2="14.0335" y2="10.0135" width="0" layer="19" extent="1-1"/>
+<wire x1="22.352" y1="9.359" x2="18.534" y2="7.512" width="0" layer="19" extent="1-1"/>
+<wire x1="1.27" y1="6.35" x2="14.0335" y2="10.0135" width="0" layer="19" extent="1-1"/>
 </signal>
 <signal name="3.3V">
@@
 <wire x1="13.843" y1="12.7" x2="16.3195" y2="12.7" width="0.254" layer="1"/>
 <wire x1="12.7" y1="13.843" x2="13.843" y2="12.7" width="0.254" layer="1"/>
-<wire x1="19.685" y1="9.906" x2="19.431" y2="10.16" width="0.254" layer="1"/>
-<wire x1="19.431" y1="10.16" x2="16.593" y2="10.16" width="0.254" layer="1"/>
-<wire x1="16.593" y1="10.16" x2="16.3195" y2="9.8865" width="0.254" layer="1"/>
-<wire x1="19.685" y1="9.906" x2="19.685" y2="8.128" width="0.254" layer="1"/>
+<wire x1="16.3195" y1="9.8865" x2="16.593" y2="10.16" width="0.254" layer="1"/>
 <wire x1="16.3195" y1="15.5135" x2="16.466" y2="15.367" width="0.254" layer="1"/>
 <wire x1="16.466" y1="15.367" x2="20.066" y2="15.367" width="0.254" layer="1"/>
-<wire x1="20.066" y1="15.367" x2="20.934" y2="16.235" width="0.254" layer="1"/>
-<wire x1="20.934" y1="16.235" x2="20.934" y2="16.275" width="0.254" layer="1"/>
 <contactref element="C4" pad="1"/>
 <contactref element="U$2" pad="P5"/>
 <contactref element="C7" pad="1"/>
-<wire x1="19.685" y1="8.128" x2="20.193" y2="7.62" width="0.254" layer="1"/>
-<wire x1="20.826" y1="7.62" x2="20.934" y2="7.512" width="0.254" layer="1"/>
-<wire x1="20.193" y1="7.62" x2="20.826" y2="7.62" width="0.254" layer="1"/>
 <wire x1="22.352" y1="7.659" x2="22.205" y2="7.512" width="0.254" layer="1"/>
-<wire x1="22.205" y1="7.512" x2="20.934" y2="7.512" width="0.254" layer="1"/>
-<wire x1="20.934" y1="16.275" x2="21.081" y2="16.422" width="0.254" layer="1"/>
-<wire x1="21.081" y1="16.422" x2="22.352" y2="16.422" width="0.254" layer="1"/>
 <wire x1="15.379" y1="23.622" x2="14.097" y2="23.622" width="0.254" layer="1"/>
 <wire x1="14.097" y1="23.622" x2="13.208" y2="24.511" width="0.254" layer="1"/>
@@
 <wire x1="17.526" y1="23.583" x2="15.418" y2="23.583" width="0.254" layer="1"/>
 <wire x1="15.418" y1="23.583" x2="15.379" y2="23.622" width="0.254" layer="1"/>
+<wire x1="19.81505" y1="9.412" x2="20.934" y2="9.412" width="0.254" layer="1"/>
+<wire x1="19.06705" y1="10.16" x2="19.81505" y2="9.412" width="0.254" layer="1"/>
+<wire x1="16.593" y1="10.16" x2="19.06705" y2="10.16" width="0.254" layer="1"/>
+<wire x1="20.662" y1="19.685" x2="20.934" y2="18.175" width="0" layer="19" extent="1-1"/>
+<wire x1="20.066" y1="15.367" x2="20.934" y2="18.175" width="0" layer="19" extent="1-1"/>
+<wire x1="22.352" y1="7.659" x2="20.934" y2="9.412" width="0" layer="19" extent="1-1"/>
 </signal>
 <signal name="N$2">
@@
 <contactref element="U$1" pad="P4"/>
 <contactref element="J2" pad="1"/>
-<wire x1="20.934" y1="18.817" x2="20.574" y2="19.177" width="0.254" layer="1"/>
-<via x="20.574" y="19.177" extent="1-16" drill="0.381"/>
 <wire x1="24.13" y1="13.97" x2="23.368" y2="13.97" width="0.254" layer="16"/>
-<wire x1="23.368" y1="13.97" x2="20.574" y2="16.764" width="0.254" layer="16"/>
-<wire x1="20.574" y1="16.764" x2="20.574" y2="19.177" width="0.254" layer="16"/>
-<wire x1="20.934" y1="18.175" x2="20.934" y2="18.817" width="0.254" layer="1"/>
+<wire x1="23.368" y1="13.97" x2="20.934" y2="16.275" width="0" layer="19" extent="1-16"/>
 </signal>
 <signal name="DIR_OUT">
 <contactref element="U$2" pad="P4"/>
 <contactref element="J2" pad="2"/>
-<wire x1="24.13" y1="11.43" x2="22.606" y2="11.43" width="0.254" layer="1"/>
-<wire x1="20.934" y1="9.758" x2="22.606" y2="11.43" width="0.254" layer="1"/>
-<wire x1="20.934" y1="9.412" x2="20.934" y2="9.758" width="0.254" layer="1"/>
+<wire x1="20.934" y1="7.512" x2="24.13" y2="11.43" width="0" layer="19" extent="1-1"/>
 </signal>
 </signals>

Commit message: Removes gerbers, removes caps from schmitt trigger on both designs, adds 1uF cap to V_USB on breakout
Parts:
- moved C7 0.13 mm to (22.2, 8.51), turned to 270 degrees
Routing:
- net 3.3V: track 50.0 -> 56.2 mm
- net DIR_OUT: track 0.00 -> 5.39 mm, vias 0 -> 1
- net WT_OUT: track 0.76 -> 4.15 mm
Changed lines of the file:
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@@
 <attribute name="VALUE" value="0.1uF" x="19.812" y="20.447" size="0.6096" layer="27" font="vector" ratio="20" rot="R180" align="top-center"/>
 </element>
-<element name="C7" library="SparkFun-Capacitors" package="0603" value="0.1uF" x="22.352" y="8.509" smashed="yes" rot="R90">
-<attribute name="NAME" x="21.59" y="8.509" size="0.6096" layer="25" font="vector" ratio="20" rot="R90" align="bottom-center"/>
-<attribute name="PROD_ID" value="CAP-08390" x="22.352" y="8.509" size="1.778" layer="27" font="vector" ratio="15" rot="R90" display="off"/>
-<attribute name="VALUE" value="0.1uF" x="23.114" y="8.509" size="0.6096" layer="27" font="vector" ratio="20" rot="R90" align="top-center"/>
+<element name="C7" library="SparkFun-Capacitors" package="0603" value="0.1uF" x="22.225" y="8.509" smashed="yes" rot="R270">
+<attribute name="NAME" x="22.987" y="8.509" size="0.6096" layer="25" font="vector" ratio="20" rot="R270" align="bottom-center"/>
+<attribute name="PROD_ID" value="CAP-08390" x="22.225" y="8.509" size="1.778" layer="27" font="vector" ratio="15" rot="R270" display="off"/>
+<attribute name="VALUE" value="0.1uF" x="21.463" y="8.509" size="0.6096" layer="27" font="vector" ratio="20" rot="R270" align="top-center"/>
 </element>
 <element name="LOGO1" library="SparkFun-Aesthetics" package="SFE_LOGO_NAME_FLAME_.1" value="SFE_LOGO_NAME_FLAME.1_INCH" x="12.7" y="12.7" smashed="yes" rot="MR270"/>
@@
 <via x="15.24" y="13.97" extent="1-16" drill="0.381"/>
 <via x="15.24" y="11.557" extent="1-16" drill="0.381"/>
-<via x="19.685" y="16.256" extent="1-16" drill="0.381"/>
 <contactref element="C7" pad="2"/>
 <contactref element="U$2" pad="P3"/>
 <contactref element="C4" pad="2"/>
 <contactref element="U$1" pad="P3"/>
+<via x="17.399" y="16.129" extent="1-16" drill="0.381"/>
 </signal>
 <signal name="3.3V">
@@
 <wire x1="16.3195" y1="9.8865" x2="16.593" y2="10.16" width="0.254" layer="1"/>
 <wire x1="16.3195" y1="15.5135" x2="16.466" y2="15.367" width="0.254" layer="1"/>
-<wire x1="16.466" y1="15.367" x2="20.066" y2="15.367" width="0.254" layer="1"/>
 <contactref element="C4" pad="1"/>
 <contactref element="U$2" pad="P5"/>
 <contactref element="C7" pad="1"/>
-<wire x1="22.352" y1="7.659" x2="22.205" y2="7.512" width="0.254" layer="1"/>
 <wire x1="15.379" y1="23.622" x2="14.097" y2="23.622" width="0.254" layer="1"/>
 <wire x1="14.097" y1="23.622" x2="13.208" y2="24.511" width="0.254" layer="1"/>
@@
 <wire x1="19.06705" y1="10.16" x2="19.81505" y2="9.412" width="0.254" layer="1"/>
 <wire x1="16.593" y1="10.16" x2="19.06705" y2="10.16" width="0.254" layer="1"/>
-<wire x1="20.662" y1="19.685" x2="20.934" y2="18.175" width="0" layer="19" extent="1-1"/>
-<wire x1="20.066" y1="15.367" x2="20.934" y2="18.175" width="0" layer="19" extent="1-1"/>
-<wire x1="22.352" y1="7.659" x2="20.934" y2="9.412" width="0" layer="19" extent="1-1"/>
+<wire x1="16.3195" y1="15.5135" x2="16.593" y2="15.24" width="0.254" layer="1"/>
+<wire x1="16.593" y1="15.24" x2="19.05" y2="15.24" width="0.254" layer="1"/>
+<wire x1="19.05" y1="15.24" x2="19.685" y2="15.875" width="0.254" layer="1"/>
+<wire x1="20.08" y1="18.175" x2="20.934" y2="18.175" width="0.254" layer="1"/>
+<wire x1="19.685" y1="15.875" x2="19.685" y2="17.78" width="0.254" layer="1"/>
+<wire x1="19.685" y1="17.78" x2="20.08" y2="18.175" width="0.254" layer="1"/>
+<wire x1="20.934" y1="18.175" x2="20.662" y2="18.447" width="0.254" layer="1"/>
+<wire x1="20.662" y1="18.447" x2="20.662" y2="19.685" width="0.254" layer="1"/>
+<wire x1="20.934" y1="9.412" x2="22.172" y2="9.412" width="0.254" layer="1"/>
+<wire x1="22.172" y1="9.412" x2="22.225" y2="9.359" width="0.254" layer="1"/>
 </signal>
 <signal name="N$2">
@@
 <contactref element="U$1" pad="P4"/>
 <contactref element="J2" pad="1"/>
-<wire x1="24.13" y1="13.97" x2="23.368" y2="13.97" width="0.254" layer="16"/>
-<wire x1="23.368" y1="13.97" x2="20.934" y2="16.275" width="0" layer="19" extent="1-16"/>
+<wire x1="20.934" y1="16.275" x2="21.825" y2="16.275" width="0.254" layer="1"/>
+<wire x1="21.825" y1="16.275" x2="24.13" y2="13.97" width="0.254" layer="1"/>
 </signal>
 <signal name="DIR_OUT">
 <contactref element="U$2" pad="P4"/>
 <contactref element="J2" pad="2"/>
-<wire x1="20.934" y1="7.512" x2="24.13" y2="11.43" width="0" layer="19" extent="1-1"/>
+<wire x1="20.934" y1="7.512" x2="20.934" y2="8.488" width="0.254" layer="1"/>
+<wire x1="20.934" y1="8.488" x2="20.955" y2="8.509" width="0.254" layer="1"/>
+<via x="20.955" y="8.509" extent="1-16" drill="0.381"/>
+<wire x1="20.955" y1="8.509" x2="23.876" y2="11.43" width="0.254" layer="16"/>
+<wire x1="23.876" y1="11.43" x2="24.13" y2="11.43" width="0.254" layer="16"/>
 </signal>
 </signals>

Commit message: Updates wheel tick and direction circuitry with correct grounding
Parts:
- removed C2, C3: 22nF, SparkFun-Capacitors:0603
Connections:
- net DIR_SCHMITT: no longer C3.1
- net GND: no longer C2.2, C3.2
- net WT_SCHMITT: no longer C2.1
Routing:
- net DIR_SCHMITT: track 21.7 -> 20.5 mm
- net WT_SCHMITT: track 12.6 -> 11.5 mm
Changed lines of the file:
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@@
 <attribute name="VALUE" x="9.3345" y="10.541" size="0.6096" layer="27" font="vector" ratio="20" rot="R90" align="top-center"/>
-</element>
-<element name="C2" library="SparkFun-Capacitors" package="0603" value="22nF" x="14.1605" y="16.3635" smashed="yes" rot="R270">
-<attribute name="NAME" x="14.9225" y="16.3635" size="0.6096" layer="25" font="vector" ratio="20" rot="R270" align="bottom-center"/>
-<attribute name="PROD_ID" value="CAP-07885" x="14.1605" y="16.3635" size="1.778" layer="27" font="vector" ratio="15" rot="R270" display="off"/>
-<attribute name="VALUE" x="13.3985" y="16.3635" size="0.6096" layer="27" font="vector" ratio="20" rot="R270" align="top-center"/>
-</element>
-<element name="C3" library="SparkFun-Capacitors" package="0603" value="22nF" x="14.0335" y="9.1635" smashed="yes" rot="R90">
-<attribute name="NAME" x="13.2715" y="9.1635" size="0.6096" layer="25" font="vector" ratio="20" rot="R90" align="bottom-center"/>
-<attribute name="PROD_ID" value="CAP-07885" x="14.0335" y="9.1635" size="1.778" layer="27" font="vector" ratio="15" rot="R90" display="off"/>
-<attribute name="VALUE" x="14.7955" y="9.1635" size="0.6096" layer="27" font="vector" ratio="20" rot="R90" align="top-center"/>
 </element>
 <element name="C6" library="SparkFun-Capacitors" package="0603" value="1nF" x="8.5725" y="14.351" smashed="yes" rot="R270">
@@
 <contactref element="U1" pad="P5"/>
 <contactref element="C5" pad="2"/>
-<contactref element="C2" pad="2"/>
-<contactref element="C3" pad="2"/>
 <contactref element="J1" pad="1"/>
 <polygon width="0.254" layer="1" isolate="0.254">
@@
 <contactref element="U$1" pad="P2"/>
 <contactref element="R3" pad="1"/>
-<contactref element="C2" pad="1"/>
-<wire x1="14.1605" y1="17.2135" x2="15.24" y2="17.2135" width="0.254" layer="1"/>
 <wire x1="15.24" y1="17.2135" x2="16.3195" y2="17.2135" width="0.254" layer="1"/>
 <wire x1="14.097" y1="18.542" x2="14.732" y2="18.542" width="0.254" layer="1"/>
@@
 <contactref element="U$2" pad="P2"/>
 <contactref element="R6" pad="1"/>
-<contactref element="C3" pad="1"/>
 <wire x1="18.534" y1="8.462" x2="16.595" y2="8.462" width="0.254" layer="1"/>
 <wire x1="16.595" y1="8.462" x2="16.3195" y2="8.1865" width="0.254" layer="1"/>
 <wire x1="16.3195" y1="8.1865" x2="16.1925" y2="8.3135" width="0.254" layer="1"/>
 <wire x1="16.1925" y1="8.3135" x2="15.24" y2="8.3135" width="0.254" layer="1"/>
-<wire x1="15.24" y1="8.3135" x2="14.0335" y2="8.3135" width="0.254" layer="1"/>
 <via x="13.97" y="20.447" extent="1-16" drill="0.381"/>
 <wire x1="13.97" y1="7.874" x2="13.97" y2="20.447" width="0.254" layer="16"/>
